Commit message: Added some links and joints so that the xtion sensor can be linked into the model.  WIP, a lot is still hard-coded

File: kobayashi_maru_description/urdf/kobayashi_maru_model.urdf.xacro (robot description, xacro)
@@ -1,5 +1,27 @@
 <?xml version="1.0"?>
-<robot xmlns:xacro="http://www.ros.org/wiki/xacro">
-	<xacro:include filename="$(find ackermann_vehicle_description)/urdf/em_3905.urdf.xacro" />
-	<xacro:include filename="$(find hector_sensors_description)/urdf/asus_camera.urdf.xacro" />
+<robot name="myfirst" xmlns:xacro="http://www.ros.org/wiki/xacro">
+  <xacro:include filename="$(find ackermann_vehicle_description)/urdf/em_3905.urdf.xacro" />
+  <xacro:include filename="$(find hector_sensors_description)/urdf/asus_camera.urdf.xacro" parent="pan_base"/>
+  <!-- Pan Base -->
+  <link name="pan_base">
+    <visual>
+      <geometry>
+	<cylinder length="0.0460375" radius="0.0492125"/>
+      </geometry>
+      <material name="tire_mat"/>
+    </visual>
+    <collision>
+      <geometry>
+	<cylinder length="0.0460375" radius="0.0492125"/>
+      </geometry>
+    </collision>
+  </link>
+  <joint name="chassis_to_pan_base" type="fixed">
+    <parent link="chassis"/>
+    <child link="pan_base"/>
+    <origin xyz="0 0 .2"/>
+  </joint>
+  <xacro:asus_camera name="xtion" parent="pan_base">
+    <origin xyz="0.0 0.0 0.0460375" rpy="0 0.3926990 0"/>
+  </xacro:asus_camera>
 </robot>
